File: split70kb.kicad_pcb (KiCad board)
At the start: 2 copper layers, 194.7 x 143.9 mm, 88 parts, among them J1 USB_C_Receptacle_USB2.0, J2 AudioJack4, K1 KEYSW, K10 KEYSW, K11 KEYSW, K12 KEYSW, K13 KEYSW, K14 KEYSW, K15 KEYSW, K16 KEYSW, K17 KEYSW, K18 KEYSW, K19 KEYSW, K2 KEYSW, K20 KEYSW, K21 KEYSW, K22 KEYSW, K23 KEYSW, K24 KEYSW, K25 KEYSW, K27 KEYSW, K28 KEYSW, K29 KEYSW, K3 KEYSW, K30 KEYSW, K31 KEYSW, K32 KEYSW, K33 KEYSW, K34 KEYSW, K35 KEYSW, K4 KEYSW, K5 KEYSW, K6 KEYSW, K7 KEYSW, K8 KEYSW, K9 KEYSW, SW1 SW_PUSH, U1 ATMEGA32U4, X1 XTAL_GND

Commit message: update for right side too in one board
Parts:
- removed C1, C2: 22p, Capacitor_SMD:C_0805_2012Metric
- removed C3, C4, C5, C6, C7: 0.1u, Capacitor_SMD:C_0805_2012Metric
- removed C8: 1u, Capacitor_SMD:C_0805_2012Metric
- removed R1, R2: 10k, Resistor_SMD:R_0805_2012Metric
- removed R3, R4: 22, Resistor_SMD:R_0805_2012Metric
- removed R5, R6: 5.1K, Resistor_SMD:R_0805_2012Metric
- removed SW1: SW_PUSH, Button_Switch_SMD:SW_SPST_TL3342
- removed X1: XTAL_GND, Crystal:Crystal_SMD_SeikoEpson_FA238-4Pin_3.2x2.5mm
- added D36: D, keyboard_parts.pretty-master:D_SOD123_axial, F.Cu at (339.2, 133.3)
- added D37: D, keyboard_parts.pretty-master:D_SOD123_axial, F.Cu at (339.2, 114.2)
- added D38: D, keyboard_parts.pretty-master:D_SOD123_axial, F.Cu at (339.0, 95.2)
- added D39: D, keyboard_parts.pretty-master:D_SOD123_axial, F.Cu at (339.1, 76.0)
- added D40: D, keyboard_parts.pretty-master:D_SOD123_axial, F.Cu at (339.0, 57.2)
- added D41: D, keyboard_parts.pretty-master:D_SOD123_axial, F.Cu at (320.2, 138.1)
- added D42: D, keyboard_parts.pretty-master:D_SOD123_axial, F.Cu at (320.1, 119.0)
- added D43: D, keyboard_parts.pretty-master:D_SOD123_axial, F.Cu at (320.1, 99.9)
- added D44: D, keyboard_parts.pretty-master:D_SOD123_axial, F.Cu at (320.2, 80.9)
- added D45: D, keyboard_parts.pretty-master:D_SOD123_axial, F.Cu at (319.9, 61.9)
- added D46: D, keyboard_parts.pretty-master:D_SOD123_axial, F.Cu at (301.0, 104.7)
- added D47: D, keyboard_parts.pretty-master:D_SOD123_axial, F.Cu at (301.0, 123.7)
- added D48: D, keyboard_parts.pretty-master:D_SOD123_axial, F.Cu at (301.0, 142.7)
- added D49: D, keyboard_parts.pretty-master:D_SOD123_axial, F.Cu at (300.9, 85.8)
- added D50: D, keyboard_parts.pretty-master:D_SOD123_axial, F.Cu at (301.0, 66.6)
- added D51: D, keyboard_parts.pretty-master:D_SOD123_axial, F.Cu at (282.0, 142.7)
- added D52: D, keyboard_parts.pretty-master:D_SOD123_axial, F.Cu at (281.9, 123.7)
- added D53: D, keyboard_parts.pretty-master:D_SOD123_axial, F.Cu at (282.2, 104.9)
- added D54: D, keyboard_parts.pretty-master:D_SOD123_axial, F.Cu at (282.1, 85.6)
- added D55: D, keyboard_parts.pretty-master:D_SOD123_axial, F.Cu at (282.0, 66.6)
- added D56: D, keyboard_parts.pretty-master:D_SOD123_axial, F.Cu at (262.9, 138.1)
- added D57: D, keyboard_parts.pretty-master:D_SOD123_axial, F.Cu at (262.9, 118.9)
- added D58: D, keyboard_parts.pretty-master:D_SOD123_axial, F.Cu at (263.0, 99.8)
- added D59: D, keyboard_parts.pretty-master:D_SOD123_axial, F.Cu at (263.0, 80.7)
- added D60: D, keyboard_parts.pretty-master:D_SOD123_axial, F.Cu at (263.0, 61.7)
- added D61: D, keyboard_parts.pretty-master:D_SOD123_axial, F.Cu at (243.8, 133.2)
- added D62: D, keyboard_parts.pretty-master:D_SOD123_axial, F.Cu at (243.9, 114.2)
- added D63: D, keyboard_parts.pretty-master:D_SOD123_axial, F.Cu at (243.9, 95.2)
- added D64: D, keyboard_parts.pretty-master:D_SOD123_axial, F.Cu at (243.9, 76.1)
- added D65: D, keyboard_parts.pretty-master:D_SOD123_axial, F.Cu at (217.3, 44.0)
- added D66: D, keyboard_parts.pretty-master:D_SOD123_axial, F.Cu at (207.7, 60.3)
- added D67: D, keyboard_parts.pretty-master:D_SOD123_axial, F.Cu at (198.5, 76.5)
- added D68: D, keyboard_parts.pretty-master:D_SOD123_axial, F.Cu at (182.2, 67.1)
- added D69: D, keyboard_parts.pretty-master:D_SOD123_axial, F.Cu at (191.7, 50.9)
- added D70: D, keyboard_parts.pretty-master:D_SOD123_axial, F.Cu at (200.9, 34.6)
- added K26: KEYSW, keyboard_parts.pretty-master:Mx_Alps_100, F.Cu at (128.6, 43.9)
- added K36: KEYSW, keyboard_parts.pretty-master:Mx_Alps_100, B.Cu at (339.1, 137.6)
- added K37: KEYSW, keyboard_parts.pretty-master:Mx_Alps_100, B.Cu at (339.1, 118.5)
- added K38: KEYSW, keyboard_parts.pretty-master:Mx_Alps_100, B.Cu at (339.1, 99.4)
- added K39: KEYSW, keyboard_parts.pretty-master:Mx_Alps_100, B.Cu at (339.1, 80.3)
- added K40: KEYSW, keyboard_parts.pretty-master:Mx_Alps_100, B.Cu at (339.1, 61.3)
- added K41: KEYSW, keyboard_parts.pretty-master:Mx_Alps_100, B.Cu at (320.1, 142.3)
- added K42: KEYSW, keyboard_parts.pretty-master:Mx_Alps_100, B.Cu at (320.1, 123.2)
- added K43: KEYSW, keyboard_parts.pretty-master:Mx_Alps_100, B.Cu at (320.0, 104.2)
- added K44: KEYSW, keyboard_parts.pretty-master:Mx_Alps_100, B.Cu at (320.1, 85.1)
- added K45: KEYSW, keyboard_parts.pretty-master:Mx_Alps_100, B.Cu at (320.1, 66.1)
- added K46: KEYSW, keyboard_parts.pretty-master:Mx_Alps_100, B.Cu at (301.0, 147.0)
- added K47: KEYSW, keyboard_parts.pretty-master:Mx_Alps_100, B.Cu at (301.0, 128.0)
- added K48: KEYSW, keyboard_parts.pretty-master:Mx_Alps_100, B.Cu at (301.0, 108.9)
- added K49: KEYSW, keyboard_parts.pretty-master:Mx_Alps_100, B.Cu at (301.0, 90.0)
- added K50: KEYSW, keyboard_parts.pretty-master:Mx_Alps_100, B.Cu at (301.0, 70.8)
- added K51: KEYSW, keyboard_parts.pretty-master:Mx_Alps_100, B.Cu at (282.0, 147.0)
- added K52: KEYSW, keyboard_parts.pretty-master:Mx_Alps_100, B.Cu at (281.9, 128.0)
- added K53: KEYSW, keyboard_parts.pretty-master:Mx_Alps_100, B.Cu at (281.9, 109.0)
- added K54: KEYSW, keyboard_parts.pretty-master:Mx_Alps_100, B.Cu at (282.0, 89.8)
- added K55: KEYSW, keyboard_parts.pretty-master:Mx_Alps_100, B.Cu at (281.9, 70.8)
- added K56: KEYSW, keyboard_parts.pretty-master:Mx_Alps_100, B.Cu at (262.9, 142.3)
- added K57: KEYSW, keyboard_parts.pretty-master:Mx_Alps_100, B.Cu at (262.9, 123.2)
- added K58: KEYSW, keyboard_parts.pretty-master:Mx_Alps_100, B.Cu at (262.9, 104.2)
- added K59: KEYSW, keyboard_parts.pretty-master:Mx_Alps_100, B.Cu at (262.9, 85.1)
- added K60: KEYSW, keyboard_parts.pretty-master:Mx_Alps_100, B.Cu at (262.9, 66.1)
- added K61: KEYSW, keyboard_parts.pretty-master:Mx_Alps_100, B.Cu at (243.8, 137.5)
- added K62: KEYSW, keyboard_parts.pretty-master:Mx_Alps_100, B.Cu at (243.8, 118.5)
- added K63: KEYSW, keyboard_parts.pretty-master:Mx_Alps_100, B.Cu at (243.9, 99.4)
- added K64: KEYSW, keyboard_parts.pretty-master:Mx_Alps_100, B.Cu at (243.9, 80.4)
- added K65: KEYSW, keyboard_parts.pretty-master:Mx_Alps_100, B.Cu at (215.1, 47.7)
- added K66: KEYSW, keyboard_parts.pretty-master:Mx_Alps_100, B.Cu at (205.7, 64.0)
- added K67: KEYSW, keyboard_parts.pretty-master:Mx_Alps_100, B.Cu at (196.3, 80.3)
- added K68: KEYSW, keyboard_parts.pretty-master:Mx_Alps_100, B.Cu at (180.1, 70.9)
- added K69: KEYSW, keyboard_parts.pretty-master:Mx_Alps_100, B.Cu at (189.5, 54.6)
- added K70: KEYSW, keyboard_parts.pretty-master:Mx_Alps_100, B.Cu at (198.9, 38.3)
- added U2: ProMicro, keyboard_parts.pretty-master:Pro_Micro, B.Cu at (147.9, 37.1)
- J1: value USB_C_Receptacle_USB2.0 -> AudioJack4; footprint Connector_USB:USB_C_Receptacle_Molex_105450-0101 -> Connector_Audio:Jack_3.5mm_PJ320D_Horizontal; moved to F.Cu
- U1: value ATMEGA32U4 -> ProMicro; footprint Package_QFP:TQFP-44_10x10mm_P0.8mm -> keyboard_parts.pretty-master:Pro_Micro; moved to F.Cu
- moved J1 105.9 mm to (207.2, 93.1), turned to 60 degrees
- moved U1 91.6 mm to (224.8, 145.8)
- moved K33 3.44 mm to (194.3, 112.3)
- moved D14 3.44 mm to (71.1, 95.9)
- moved K14 3.44 mm to (71.2, 91.7)
- moved D24 3.44 mm to (109.1, 100.5)
- moved K27 3.44 mm to (128.3, 63.3)
- moved D25 3.44 mm to (109.3, 119.7)
- moved D28 3.44 mm to (128.3, 86.6)
- moved D26 3.44 mm to (128.7, 48.3)
- moved K28 3.44 mm to (128.3, 82.1)
- moved D33 3.44 mm to (192.0, 115.8)
- moved K31 3.44 mm to (168.7, 119.2)
- moved D17 3.44 mm to (90.2, 57.7)
- moved D29 3.44 mm to (128.3, 105.3)
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Connections:
- U1 pad 10: unconnected-(U1-PB2/MOSI-Pad10) -> rcol1
- U1 pad 11: unconnected-(U1-PB3/MISO-Pad11) -> rcol2
- U1 pad 12: unconnected-(U1-PB7/~{RTS}-Pad12) -> rcol3
- U1 pad 13: Net-(U1-~{RESET}) -> unconnected-(U1-B6-Pad13)
- U1 pad 16: Net-(U1-XTAL1) -> unconnected-(U1-B1-Pad16)
- U1 pad 17: Net-(U1-XTAL2) -> rcol5
- U1 pad 18: unconnected-(U1-PD0/INT0-Pad18) -> rcol5
- U1 pad 19: unconnected-(U1-PD1/INT1-Pad19) -> rcol5
- U1 pad 2: unconnected-(U1-UVcc-Pad2) -> rpd2
- U1 pad 20: pd2 -> rcol4
- U1 pad 21: unconnected-(U1-PD3/TXD1-Pad21) -> +3.3V
- U1 pad 23: GND -> GND1
- U1 pad 24: VCC -> unconnected-(U1-RAW-Pad24)
- U1 pad 3: Net-(U1-D-) -> GND1
- U1 pad 4: Net-(U1-D+) -> GND1
- U1 pad 5: GND -> rcol5
- U1 pad 6: Net-(U1-UCap) -> rcol5
- U1 pad 7: VCC -> rcol5
- U1 pad 8: unconnected-(U1-PB0/SS-Pad8) -> rcol5
- U1 pad 9: unconnected-(U1-PB1/SCK-Pad9) -> rcol5
Routing:
- net col5: track 0.00 -> 922.1 mm
- net rcol5: track 0.00 -> 918.7 mm
- net col1: track 0.00 -> 213.2 mm
- net col2: track 0.00 -> 197.3 mm
- net rcol2: track 0.00 -> 181.9 mm
- net col3: track 0.00 -> 175.0 mm
- net rcol1: track 0.00 -> 168.7 mm
- net rcol3: track 0.00 -> 144.5 mm
- net col4: track 0.00 -> 140.3 mm
- net rcol4: track 0.00 -> 127.6 mm
- net rpd2: track 0.00 -> 88.9 mm, vias 0 -> 1
- net GND: track 0.00 -> 88.7 mm
- net GND1: track 0.00 -> 72.8 mm, vias 0 -> 1
- net pd2: track 0.00 -> 70.6 mm
- net Net-(D46-A): track 0.00 -> 61.7 mm
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- removed copper zone on B.Cu, net GND
- removed copper zone on F.Cu, net GND
Other:
- board size 194.7 x 143.9 mm -> 335.9 x 145.9 mm
