File: pcbsrc/split70kb.kicad_sch (KiCad schematic)
At the start: 144 parts, among them J1 AudioJack4, J2 AudioJack4, K1 KEYSW, K10 KEYSW, K11 KEYSW, K12 KEYSW, K13 KEYSW, K14 KEYSW, K15 KEYSW, K16 KEYSW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

Commit message: cleanup and shit
Parts:
- D1, D10, D11, D12, D13, D14, D15, D16, D17, D18, D19, D2, D20, D21, D22, D23, D24, D25, D26, D27, D28, D29, D3, D30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: JLC (none) -> 1N4148W; LCSC (none) -> C89641
